File: ESP32Prog.brd (EAGLE design)
At the start: 29.2 x 12.7 mm, 18 parts, among them T1 MMBT2222, T2 MMBT2222, U1 3.3V, U3 CH340C

Commit message: fixed gnd pin
Connections:
- net GND: now also USB_PROG.5; no longer USB_PROG.4
Changed lines of the file:
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@@
 <?xml version="1.0" encoding="utf-8"?>
 <!DOCTYPE eagle SYSTEM "eagle.dtd">
-<eagle version="9.6.1">
+<eagle version="9.6.2">
 <drawing>
 <settings>
@@
 <contactref element="C3" pad="2"/>
 <contactref element="U3" pad="1"/>
-<contactref element="USB_PROG" pad="4"/>
 <contactref element="SV1" pad="2"/>
 <contactref element="C4" pad="2"/>
@@
 <via x="5.55625" y="2.69875" extent="1-16" drill="0.35"/>
 <via x="6.6675" y="10.16" extent="1-16" drill="0.35"/>
+<contactref element="USB_PROG" pad="5"/>
 </signal>
 <signal name="+3V3">
